Commit message: 完成在main中启动设备可视化
完成在main中启动设备可视化，并输出物料ID：mesh的对应关系resource_model

添加物料模型管理类，遍历物料与resource_model，完成TF数据收集

File: unilabos/device_mesh/devices/opentrons_liquid_handler/macro_device.xacro (robot description, xacro)
@@ -19,5 +19,5 @@
       <visual>
         <geometry>
-          <mesh filename="file://${mesh_path}/device/opentrons_liquid_handler/meshes/ot2-0.stl"/>
+          <mesh filename="file://${mesh_path}/devices/opentrons_liquid_handler/meshes/ot2-0.stl"/>
         </geometry>
         <material name="">
@@ -28,5 +28,5 @@
         <origin rpy="0 0 0" xyz="0 0 0"/>
         <geometry>
-          <mesh filename="file://${mesh_path}/device/opentrons_liquid_handler/meshes/ot2-0.stl"/>
+          <mesh filename="file://${mesh_path}/devices/opentrons_liquid_handler/meshes/ot2-0.stl"/>
         </geometry>
       </collision>
@@ -35,5 +35,5 @@
       <visual>
         <geometry>
-          <mesh filename="file://${mesh_path}/device/opentrons_liquid_handler/meshes/ot2-1.stl"/>
+          <mesh filename="file://${mesh_path}/devices/opentrons_liquid_handler/meshes/ot2-1.stl"/>
         </geometry>
         <material name="">
@@ -44,5 +44,5 @@
         <origin rpy="0 0 0" xyz="0 0 0"/>
         <geometry>
-          <mesh filename="file://${mesh_path}/device/opentrons_liquid_handler/meshes/ot2-1.stl"/>
+          <mesh filename="file://${mesh_path}/devices/opentrons_liquid_handler/meshes/ot2-1.stl"/>
         </geometry>
       </collision>
@@ -51,5 +51,5 @@
       <visual>
         <geometry>
-          <mesh filename="file://${mesh_path}/device/opentrons_liquid_handler/meshes/ot2-2.stl"/>
+          <mesh filename="file://${mesh_path}/devices/opentrons_liquid_handler/meshes/ot2-2.stl"/>
         </geometry>
         <material name="">
@@ -60,5 +60,5 @@
         <origin rpy="0 0 0" xyz="0 0 0"/>
         <geometry>
-          <mesh filename="file://${mesh_path}/device/opentrons_liquid_handler/meshes/ot2-2.stl"/>
+          <mesh filename="file://${mesh_path}/devices/opentrons_liquid_handler/meshes/ot2-2.stl"/>
         </geometry>
       </collision>
@@ -67,5 +67,5 @@
       <visual>
         <geometry>
-          <mesh filename="file://${mesh_path}/device/opentrons_liquid_handler/meshes/ot2-3a.stl"/>
+          <mesh filename="file://${mesh_path}/devices/opentrons_liquid_handler/meshes/ot2-3a.stl"/>
         </geometry>
         <material name="">
@@ -76,5 +76,5 @@
         <origin rpy="0 0 0" xyz="0 0 0"/>
         <geometry>
-          <mesh filename="file://${mesh_path}/device/opentrons_liquid_handler/meshes/ot2-3a.stl"/>
+          <mesh filename="file://${mesh_path}/devices/opentrons_liquid_handler/meshes/ot2-3a.stl"/>
         </geometry>
       </collision>
@@ -83,5 +83,5 @@
       <visual>
         <geometry>
-          <mesh filename="file://${mesh_path}/device/opentrons_liquid_handler/meshes/ot2-3b.stl"/>
+          <mesh filename="file://${mesh_path}/devices/opentrons_liquid_handler/meshes/ot2-3b.stl"/>
         </geometry>
         <material name="">
@@ -92,5 +92,5 @@
         <origin rpy="0 0 0" xyz="0 0 0"/>
         <geometry>
-          <mesh filename="file://${mesh_path}/device/opentrons_liquid_handler/meshes/ot2-3b.stl"/>
+          <mesh filename="file://${mesh_path}/devices/opentrons_liquid_handler/meshes/ot2-3b.stl"/>
         </geometry>
       </collision>

File: unilabos/device_mesh/devices/slide_w140/macro_device.xacro (robot description, xacro)
@@ -31,5 +31,5 @@
         <origin rpy="0 0 0" xyz="0 0 0"/>
         <geometry>
-          <mesh filename="file://${mesh_path}/device/slide_w140/meshes/base_link.STL"/>
+          <mesh filename="file://${mesh_path}/devices/slide_w140/meshes/base_link.STL"/>
         </geometry>
         <material name="">
@@ -40,5 +40,5 @@
         <origin rpy="0 0 0" xyz="0 0 0"/>
         <geometry>
-          <mesh filename="file://${mesh_path}/device/slide_w140/meshes/base_link.STL"/>
+          <mesh filename="file://${mesh_path}/devices/slide_w140/meshes/base_link.STL"/>
         </geometry>
       </collision>
@@ -53,5 +53,5 @@
         <origin rpy="0 0 0" xyz="0 0 0"/>
         <geometry>
-          <mesh filename="file://${mesh_path}/device/slide_w140/meshes/slider.STL" />
+          <mesh filename="file://${mesh_path}/devices/slide_w140/meshes/slider.STL" />
         </geometry>
         <material name="">
@@ -62,5 +62,5 @@
         <origin rpy="0 0 0" xyz="0 0 0"/>
         <geometry>
-          <mesh filename="file://${mesh_path}/device/slide_w140/meshes/slider.STL" />
+          <mesh filename="file://${mesh_path}/devices/slide_w140/meshes/slider.STL" />
         </geometry>
       </collision>
@@ -82,5 +82,5 @@
         <origin rpy="0 0 0" xyz="0 0 0"/>
         <geometry>
-          <mesh filename="file://${mesh_path}/device/slide_w140/meshes/length.STL" scale="${(length + min_d + max_d + slider_d)} 1 1"/>
+          <mesh filename="file://${mesh_path}/devices/slide_w140/meshes/length.STL" scale="${(length + min_d + max_d + slider_d)} 1 1"/>
         </geometry>
         <material name="">
@@ -91,5 +91,5 @@
         <origin rpy="0 0 0" xyz="0 0 0"/>
         <geometry>
-          <mesh filename="file://${mesh_path}/device/slide_w140/meshes/length.STL" scale="${(length + min_d + max_d + slider_d)} 1 1"/>
+          <mesh filename="file://${mesh_path}/devices/slide_w140/meshes/length.STL" scale="${(length + min_d + max_d + slider_d)} 1 1"/>
         </geometry>
       </collision>
@@ -109,5 +109,5 @@
         <origin rpy="0 0 0" xyz="0 0 0"/>
         <geometry>
-          <mesh filename="file://${mesh_path}/device/slide_w140/meshes/slide_end.STL"/>
+          <mesh filename="file://${mesh_path}/devices/slide_w140/meshes/slide_end.STL"/>
         </geometry>
         <material name="">
@@ -118,5 +118,5 @@
         <origin rpy="0 0 0" xyz="0 0 0"/>
         <geometry>
-          <mesh filename="file://${mesh_path}/device/slide_w140/meshes/slide_end.STL"/>
+          <mesh filename="file://${mesh_path}/devices/slide_w140/meshes/slide_end.STL"/>
         </geometry>
       </collision>

Commit message: 修改模型方向，在yaml中添加变换属性

File: unilabos/device_mesh/devices/opentrons_liquid_handler/macro_device.xacro (robot description, xacro)
@@ -5,5 +5,5 @@
     <joint name="${station_name}${device_name}base_link_joint" type="fixed">
       <origin xyz="${x} ${y} ${z}" rpy="0 0 ${r}" />
-      <parent link="${station_name}${device_name}${parent_link}"/>
+      <parent link="${parent_link}"/>
       <child link="${station_name}${device_name}device_link"/>
       <axis xyz="0 0 0"/>
@@ -11,5 +11,5 @@
     <link name="${station_name}${device_name}device_link"/>
     <joint name="${station_name}${device_name}device_link_joint" type="fixed">
-      <origin xyz="-0.31 0.28 0" rpy="0 0 0" />
+      <origin xyz="-0.11565 0.496 0" rpy="0 0 0" />
       <parent link="${station_name}${device_name}device_link"/>
       <child link="${station_name}${device_name}main_link"/>
