Commit message: change arm's name

File: unilabos/device_mesh/devices/arm_slider/config/macro.ros2_control.xacro (robot description, xacro)
@@ -1,7 +1,7 @@
 <?xml version="1.0"?>
 <robot xmlns:xacro="http://www.ros.org/wiki/xacro">
-    <xacro:macro name="benyao_arm_ros2_control" params="device_name mesh_path">
-        <xacro:property name="initial_positions" value="${load_yaml(mesh_path + '/devices/benyao_arm/config/initial_positions.yaml')['initial_positions']}"/>
-        <ros2_control name="${device_name}benyao_arm" type="system">
+    <xacro:macro name="arm_slider_ros2_control" params="device_name mesh_path">
+        <xacro:property name="initial_positions" value="${load_yaml(mesh_path + '/devices/arm_slider/config/initial_positions.yaml')['initial_positions']}"/>
+        <ros2_control name="${device_name}arm_slider" type="system">
             <hardware>
                 <!-- By default, set up controllers for simulation. This won't work on real hardware -->

File: unilabos/device_mesh/devices/arm_slider/config/macro.srdf.xacro (robot description, xacro)
@@ -5,5 +5,5 @@
 -->
 <robot xmlns:xacro="http://ros.org/wiki/xacro">
-    <xacro:macro name="benyao_arm_srdf" params="device_name">
+    <xacro:macro name="arm_slider_srdf" params="device_name">
         <!--GROUPS: Representation of a set of joints and links. This can be useful for specifying DOF to plan for, defining arms, end effectors, etc-->
         <!--LINKS: When a link is specified, the parent joint of that link (if it exists) is automatically included-->

File: unilabos/device_mesh/devices/arm_slider/macro_device.xacro (robot description, xacro)
@@ -1,7 +1,7 @@
 <?xml version="1.0" ?>
-<robot xmlns:xacro="http://ros.org/wiki/xacro" name="benyao_arm">
-  <xacro:macro name="benyao_arm" params="mesh_path:='' parent_link:='' station_name:='' device_name:='' x:=0 y:=0 z:=0 rx:=0 ry:=0 r:=0">
+<robot xmlns:xacro="http://ros.org/wiki/xacro" name="arm_slider">
+  <xacro:macro name="arm_slider" params="mesh_path:='' parent_link:='' station_name:='' device_name:='' x:=0 y:=0 z:=0 rx:=0 ry:=0 r:=0">
     <!-- Read .yaml files from disk, load content into properties -->
-    <xacro:property name= "joint_limit_parameters" value="${xacro.load_yaml(mesh_path + '/devices/benyao_arm/joint_limit.yaml')}"/>
+    <xacro:property name= "joint_limit_parameters" value="${xacro.load_yaml(mesh_path + '/devices/arm_slider/joint_limit.yaml')}"/>
     <!-- Extract subsections from yaml dictionaries -->
     <xacro:property name= "sec_limits" value="${joint_limit_parameters['joint_limits']}"/>
@@ -36,5 +36,5 @@
         <origin rpy="0 0 0" xyz="0 0 0"/>
         <geometry>
-          <mesh filename="file://${mesh_path}/devices/benyao_arm/meshes/arm_slideway.STL"/>
+          <mesh filename="file://${mesh_path}/devices/arm_slider/meshes/arm_slideway.STL"/>
         </geometry>
         <material name="">
@@ -45,5 +45,5 @@
         <origin rpy="0 0 0" xyz="0 0 0"/>
         <geometry>
-          <mesh filename="file://${mesh_path}/devices/benyao_arm/meshes/arm_slideway.STL"/>
+          <mesh filename="file://${mesh_path}/devices/arm_slider/meshes/arm_slideway.STL"/>
         </geometry>
       </collision>
@@ -69,14 +69,14 @@
         <origin rpy="0 0 0" xyz="0 0 0"/>
         <geometry>
-          <mesh filename="file://${mesh_path}/devices/benyao_arm/meshes/arm_base.STL"/>
-        </geometry>
-        <material name="">
-          <color rgba="1 1 1 1"/>
-        </material>
-      </visual>
-      <collision>
-        <origin rpy="0 0 0" xyz="0 0 0"/>
-        <geometry>
-          <mesh filename="file://${mesh_path}/devices/benyao_arm/meshes/arm_base.STL"/>
+          <mesh filename="file://${mesh_path}/devices/arm_slider/meshes/arm_base.STL"/>
+        </geometry>
+        <material name="">
+          <color rgba="1 1 1 1"/>
+        </material>
+      </visual>
+      <collision>
+        <origin rpy="0 0 0" xyz="0 0 0"/>
+        <geometry>
+          <mesh filename="file://${mesh_path}/devices/arm_slider/meshes/arm_base.STL"/>
         </geometry>
       </collision>
@@ -91,14 +91,14 @@
         <origin rpy="0 0 0" xyz="0 0 0"/>
         <geometry>
-          <mesh filename="file://${mesh_path}/devices/benyao_arm/meshes/arm_link_1.STL"/>
-        </geometry>
-        <material name="">
-          <color rgba="1 1 1 1"/>
-        </material>
-      </visual>
-      <collision>
-        <origin rpy="0 0 0" xyz="0 0 0"/>
-        <geometry>
-          <mesh filename="file://${mesh_path}/devices/benyao_arm/meshes/arm_link_1.STL"/>
+          <mesh filename="file://${mesh_path}/devices/arm_slider/meshes/arm_link_1.STL"/>
+        </geometry>
+        <material name="">
+          <color rgba="1 1 1 1"/>
+        </material>
+      </visual>
+      <collision>
+        <origin rpy="0 0 0" xyz="0 0 0"/>
+        <geometry>
+          <mesh filename="file://${mesh_path}/devices/arm_slider/meshes/arm_link_1.STL"/>
         </geometry>
       </collision>
@@ -124,14 +124,14 @@
         <origin rpy="0 0 0" xyz="0 0 0"/>
         <geometry>
-          <mesh filename="file://${mesh_path}/devices/benyao_arm/meshes/arm_link_2.STL"/>
-        </geometry>
-        <material name="">
-          <color rgba="1 1 1 1"/>
-        </material>
-      </visual>
-      <collision>
-        <origin rpy="0 0 0" xyz="0 0 0"/>
-        <geometry>
-          <mesh filename="file://${mesh_path}/devices/benyao_arm/meshes/arm_link_2.STL"/>
+          <mesh filename="file://${mesh_path}/devices/arm_slider/meshes/arm_link_2.STL"/>
+        </geometry>
+        <material name="">
+          <color rgba="1 1 1 1"/>
+        </material>
+      </visual>
+      <collision>
+        <origin rpy="0 0 0" xyz="0 0 0"/>
+        <geometry>
+          <mesh filename="file://${mesh_path}/devices/arm_slider/meshes/arm_link_2.STL"/>
         </geometry>
       </collision>
@@ -157,14 +157,14 @@
         <origin rpy="0 0 0" xyz="0 0 0"/>
         <geometry>
-          <mesh filename="file://${mesh_path}/devices/benyao_arm/meshes/arm_link_3.STL"/>
-        </geometry>
-        <material name="">
-          <color rgba="1 1 1 1"/>
-        </material>
-      </visual>
-      <collision>
-        <origin rpy="0 0 0" xyz="0 0 0"/>
-        <geometry>
-          <mesh filename="file://${mesh_path}/devices/benyao_arm/meshes/arm_link_3.STL"/>
+          <mesh filename="file://${mesh_path}/devices/arm_slider/meshes/arm_link_3.STL"/>
+        </geometry>
+        <material name="">
+          <color rgba="1 1 1 1"/>
+        </material>
+      </visual>
+      <collision>
+        <origin rpy="0 0 0" xyz="0 0 0"/>
+        <geometry>
+          <mesh filename="file://${mesh_path}/devices/arm_slider/meshes/arm_link_3.STL"/>
         </geometry>
       </collision>
@@ -190,14 +190,14 @@
         <origin rpy="0 0 0" xyz="0 0 0"/>
         <geometry>
-          <mesh filename="file://${mesh_path}/devices/benyao_arm/meshes/gripper_base.STL"/>
-        </geometry>
-        <material name="">
-          <color rgba="1 1 1 1"/>
-        </material>
-      </visual>
-      <collision>
-        <origin rpy="0 0 0" xyz="0 0 0"/>
-        <geometry>
-          <mesh filename="file://${mesh_path}/devices/benyao_arm/meshes/gripper_base.STL"/>
+          <mesh filename="file://${mesh_path}/devices/arm_slider/meshes/gripper_base.STL"/>
+        </geometry>
+        <material name="">
+          <color rgba="1 1 1 1"/>
+        </material>
+      </visual>
+      <collision>
+        <origin rpy="0 0 0" xyz="0 0 0"/>
+        <geometry>
+          <mesh filename="file://${mesh_path}/devices/arm_slider/meshes/gripper_base.STL"/>
         </geometry>
       </collision>
@@ -223,14 +223,14 @@
         <origin rpy="0 0 0" xyz="0 0 0"/>
         <geometry>
-          <mesh filename="file://${mesh_path}/devices/benyao_arm/meshes/gripper_right.STL"/>
-        </geometry>
-        <material name="">
-          <color rgba="1 1 1 1"/>
-        </material>
-      </visual>
-      <collision>
-        <origin rpy="0 0 0" xyz="0 0 0"/>
-        <geometry>
-          <mesh filename="file://${mesh_path}/devices/benyao_arm/meshes/gripper_right.STL"/>
+          <mesh filename="file://${mesh_path}/devices/arm_slider/meshes/gripper_right.STL"/>
+        </geometry>
+        <material name="">
+          <color rgba="1 1 1 1"/>
+        </material>
+      </visual>
+      <collision>
+        <origin rpy="0 0 0" xyz="0 0 0"/>
+        <geometry>
+          <mesh filename="file://${mesh_path}/devices/arm_slider/meshes/gripper_right.STL"/>
         </geometry>
       </collision>
@@ -256,5 +256,5 @@
         <origin rpy="0 3.1416 0" xyz="0 0 0"/>
         <geometry>
-          <mesh filename="file://${mesh_path}/devices/benyao_arm/meshes/gripper_left.STL"/>
+          <mesh filename="file://${mesh_path}/devices/arm_slider/meshes/gripper_left.STL"/>
         </geometry>
         <material name="">
@@ -265,5 +265,5 @@
         <origin rpy="0 3.1416 0" xyz="0 0 0"/>
         <geometry>
-          <mesh filename="file://${mesh_path}/devices/benyao_arm/meshes/gripper_left.STL"/>
+          <mesh filename="file://${mesh_path}/devices/arm_slider/meshes/gripper_left.STL"/>
         </geometry>
       </collision>
